Commit message: Working on hardware interface

File: bilbot_description/urdf/bilbot.xacro (robot description, xacro)
@@ -5,44 +5,44 @@
  	<xacro:include filename="$(find bilbot_description)/urdf/macros.xacro" />
 	<xacro:property name="PI" value="3.1415926535897931"/>
-	<xacro:property name="chassisHeight" value="0.01"/>
-	<xacro:property name="chassisLength" value="0.2"/>
-	<xacro:property name="chassisWidth" value="0.15"/>
+	<xacro:property name="chassisHeight" value="0.005"/>
+	<xacro:property name="chassisLength" value="0.185"/>
+	<xacro:property name="chassisWidth" value="0.16"/>
 	<xacro:property name="chassisMass" value="5"/>
-	<xacro:property name="layerHeight" value="0.01"/>
-	<xacro:property name="layerLength" value="0.18"/>
-	<xacro:property name="layerWidth" value="0.075"/>
-	<xacro:property name="layerMass" value="4"/>
+	<xacro:property name="layerHeight" value="0.005"/>
+	<xacro:property name="layerLength" value="0.165"/>
+	<xacro:property name="layerWidth" value="0.07"/>
+	<xacro:property name="layerMass" value=".6"/>
 	<xacro:property name="batteryHeight" value="0.027"/>
 	<xacro:property name="batteryLength" value="0.114"/>
 	<xacro:property name="batteryWidth" value="0.056"/>
-	<xacro:property name="batteryMass" value="0.423"/>
+	<xacro:property name="batteryMass" value="2"/>
 	<xacro:property name="batteryOffset" value="-0.03"/>
-	<xacro:property name="casterRadius" value="0.025"/>
-	<xacro:property name="casterMass" value="5"/>
-	<xacro:property name="wheelWidth" value="0.01"/>
-	<xacro:property name="wheelRadius" value="0.04"/>
+	<xacro:property name="casterRadius" value="0.024"/>
+	<xacro:property name="casterMass" value="2"/>
+  <xacro:property name="wheelSeparation" value="0.1875"/>
+  <xacro:property name="wheelVerticalOffset" value="0.018"/>
+	<xacro:property name="wheelWidth" value="0.008"/>
+	<xacro:property name="wheelRadius" value="0.035"/>
 	<xacro:property name="wheelPos" value="0.2"/>
-	<xacro:property name="wheelMass" value="5"/>
-	<xacro:property name="frontWidth" value="0.15"/>
-	<xacro:property name="frontLength" value="0.01"/>
-	<xacro:property name="frontHeight" value="0.075"/>
+	<xacro:property name="wheelMass" value="0.2"/>
+	<xacro:property name="frontWidth" value="0.16"/>
+	<xacro:property name="frontLength" value="0.02"/>
+	<xacro:property name="frontHeight" value="0.1"/>
 	<xacro:property name="frontMass" value="1"/>
 	<xacro:property name="motorWidth" value="0.07"/>
 	<xacro:property name="motorRadius" value="0.0125"/>
 	<xacro:property name="motorMass" value="0.104"/>
-	<xacro:property name="cameraSize" value="0.05"/>
-	<xacro:property name="cameraMass" value="0.1"/>
 	<xacro:property name="supportWidth" value="0.005"/>
-	<xacro:property name="supportHeight" value="0.03"/>
+	<xacro:property name="supportHeight" value="0.035"/>
 	<xacro:property name="supportLength" value="0.005"/>
-	<xacro:property name="supportMass" value="0.1"/>
+	<xacro:property name="supportMass" value="0.01"/>
 	<xacro:property name="raspberrypiWidth" value="0.06"/>
 	<xacro:property name="raspberrypiHeight" value="0.01"/>
 	<xacro:property name="raspberrypiLength" value="0.04"/>
-	<xacro:property name="raspberrypiMass" value="0.1"/>
+	<xacro:property name="raspberrypiMass" value="0.05"/>
 	<xacro:property name="pcbWidth" value="0.04"/>
 	<xacro:property name="pcbHeight" value="0.01"/>
 	<xacro:property name="pcbLength" value="0.04"/>
-	<xacro:property name="pcbMass" value="0.1"/>
+	<xacro:property name="pcbMass" value="0.05"/>
 	<xacro:property name="grip_shaftWidth" value="0.04"/>
 	<xacro:property name="grip_shaftRadius" value="0.005"/>
@@ -58,4 +58,12 @@
   <xacro:property name="fingerWidth" value="0.01"/>
   <xacro:property name="fingerMass" value="0.5"/>
+  <xacro:property name="cameraWidth" value="0.01"/>
+  <xacro:property name="cameraHeight" value="0.02"/>
+  <xacro:property name="cameraLength" value="0.02"/>
+  <xacro:property name="cameraMass" value="0.1"/>
+  <xacro:property name="laserWidth" value="0.01"/>
+  <xacro:property name="laserHeight" value="0.01"/>
+  <xacro:property name="laserLength" value="0.01"/>
+  <xacro:property name="laserMass" value="0.01"/>
 <link name="base_link" />
 <joint name="base_joint" type="fixed">
@@ -83,5 +91,5 @@
   </inertial>
 </link>
-<joint name="battery_joint" type="fixed">
+<!-- <joint name="battery_joint" type="fixed">
   <parent link="chassis"/>
   <child link="battery"/>
@@ -202,13 +210,113 @@
     <xacro:box_inertia m="${pcbMass}" x="${pcbLength}" y="${pcbWidth}" z="${pcbHeight}"/>
   </inertial>
-</link>
+</link> -->
 <xacro:caster fb="front" tX="1"/>
 <xacro:caster fb="back" tX="-1"/>
 <xacro:wheel lr="right" tY="1"/>
 <xacro:wheel lr="left" tY="-1"/>
-<xacro:gripper/>
+<!-- <xacro:gripper/>
 <xacro:support lr="left" fb="front" tY="1" tX="1"/>
 <xacro:support lr="right" fb="front" tY="-1" tX="1"/>
 <xacro:support lr="left" fb="back" tY="1" tX="-1"/>
 <xacro:support lr="right" fb="back" tY="-1" tX="-1"/>
+ <joint name="camera_joint" type="fixed">
+  <parent link="front"/>
+  <child link="camera"/>
+  <origin xyz="0 0 ${frontHeight}" rpy="0 0 0"/>
+</joint>
+<link name="camera">
+  <collision>
+    <origin xyz="0 0 ${cameraHeight/2}" rpy="0 0 0"/>
+    <geometry>
+      <box size="${cameraWidth} ${cameraLength} ${cameraHeight}"/>
+    </geometry>
+  </collision>
+  <visual>
+    <origin xyz="0 0 ${cameraHeight/2}" rpy="0 0 0"/>
+    <geometry>
+      <box size="${cameraWidth} ${cameraLength} ${cameraHeight}"/>
+    </geometry>
+    <material name="blue"/>
+  </visual>
+  <inertial>
+    <mass value="${cameraMass}" />
+    <origin xyz="0 0 0" rpy="0 0 0"/>
+    <box_inertia m="${cameraMass}" x="${cameraWidth}" y="${cameraLength}" z="${cameraHeight}" />
+  </inertial>
+</link>
+ <joint name="laser1_joint" type="fixed">
+    <axis xyz="0 0 0" />
+    <origin xyz="0.029 0 0.0825" rpy="0 0 0"/>
+    <parent link="front"/>
+    <child link="laser1"/>
+  </joint>
+  <link name="laser1">
+    <collision>
+      <origin xyz="0 0 0" rpy="0 0 0"/>
+      <geometry>
+    <box size="${laserWidth} ${laserLength} ${laserHeight}"/>
+      </geometry>
+    </collision>
+    <visual>
+      <origin xyz="0 0 0" rpy="0 0 0"/>
+      <geometry>
+        <box size="${laserWidth} ${laserLength} ${laserHeight}"/>
+      </geometry>
+    </visual>
+    <inertial>
+      <mass value="${laserMass}" />
+      <origin xyz="0 0 0" rpy="0 0 0"/>
+      <box_inertia m="${laserMass}" x="${laserWidth}" y="${laserLength}" z="${laserHeight}" />
+    </inertial>
+  </link>
+  <joint name="laser2_joint" type="fixed">
+    <axis xyz="0 0 0" />
+    <origin xyz="0.029 0.05 0.0825" rpy="0 0 0.261799"/>
+    <parent link="front"/>
+    <child link="laser2"/>
+  </joint>
+  <link name="laser2">
+    <collision>
+      <origin xyz="0 0 0" rpy="0 0 0"/>
+      <geometry>
+    <box size="${laserWidth} ${laserLength} ${laserHeight}"/>
+      </geometry>
+    </collision>
+    <visual>
+      <origin xyz="0 0 0" rpy="0 0 0"/>
+      <geometry>
+        <box size="${laserWidth} ${laserLength} ${laserHeight}"/>
+      </geometry>
+    </visual>
+    <inertial>
+      <mass value="${laserMass}" />
+      <origin xyz="0 0 0" rpy="0 0 0"/>
+      <box_inertia m="${laserMass}" x="${laserWidth}" y="${laserLength}" z="${laserHeight}" />
+    </inertial>
+  </link>
+  <joint name="laser3_joint" type="fixed">
+    <axis xyz="0 0 0" />
+    <origin xyz="0.029 -0.05 0.0825" rpy="0 0 -0.261799"/>
+    <parent link="front"/>
+    <child link="laser3"/>
+  </joint>
+  <link name="laser3">
+    <collision>
+      <origin xyz="0 0 0" rpy="0 0 0"/>
+      <geometry>
+    <box size="${laserWidth} ${laserLength} ${laserHeight}"/>
+      </geometry>
+    </collision>
+    <visual>
+      <origin xyz="0 0 0" rpy="0 0 0"/>
+      <geometry>
+        <box size="${laserWidth} ${laserLength} ${laserHeight}"/>
+      </geometry>
+    </visual>
+    <inertial>
+      <mass value="${laserMass}" />
+      <origin xyz="0 0 0" rpy="0 0 0"/>
+      <box_inertia m="${laserMass}" x="${laserWidth}" y="${laserLength}" z="${laserHeight}" />
+    </inertial>
+  </link> -->
 </robot>

File: bilbot_description/urdf/macros.xacro (robot description, xacro)
@@ -2,6 +2,6 @@
 <xacro:macro name="cylinder_inertia" params="m r h">
   <inertia  ixx="${m*(3*r*r+h*h)/12}" ixy = "0" ixz = "0"
-            iyy="${m*(3*r*r+h*h)/12}" iyz = "0"
-            izz="${m*r*r/2}"
+            iyy="${m*r*r/2}" iyz = "0"
+            izz="${m*(3*r*r+h*h)/12}"
   />
 </xacro:macro>
@@ -21,5 +21,5 @@
 <link name="${lr}_motor">
   <collision>
-    <origin xyz="0 0 0" rpy="-${PI/2} 0 0" />
+    <origin xyz="0 0 0" rpy="${tY*PI/2} 0 0" />
     <geometry>
       <cylinder length="${motorWidth}" radius="${motorRadius}"/>
@@ -27,5 +27,5 @@
   </collision>
   <visual>
-    <origin xyz="0 0 0" rpy="-${PI/2} 0 0" />
+    <origin xyz="0 0 0" rpy="${tY*PI/2} 0 0" />
     <geometry>
       <cylinder length="${motorWidth}" radius="${motorRadius}"/>
@@ -41,9 +41,9 @@
   <parent link="chassis"/>
   <child link="${lr}_motor"/>
-  <origin xyz="0 ${tY*((chassisWidth-motorWidth)/2+0.01)} -${motorRadius+chassisHeight/2}" />
+  <origin xyz="0 ${tY*(wheelSeparation-motorWidth-wheelWidth)/2} -${wheelVerticalOffset}" />
 </joint>
 <link name="${lr}_wheel">
   <collision>
-    <origin xyz="0 0 0" rpy="0 ${PI/2} ${PI/2}" />
+    <origin xyz="0 0 0" rpy="${tY*PI/2} 0 0" />
     <geometry>
       <cylinder length="${wheelWidth}" radius="${wheelRadius}"/>
@@ -51,5 +51,5 @@
   </collision>
   <visual>
-    <origin xyz="0 0 0" rpy="0 ${PI/2} ${PI/2}" />
+    <origin xyz="0 0 0" rpy="${tY*PI/2} 0 0" />
     <geometry>
       <cylinder length="${wheelWidth}" radius="${wheelRadius}"/>
@@ -58,17 +58,16 @@
   </visual>
   <inertial>
-    <origin xyz="0 0 0" rpy="0 ${PI/2} ${PI/2}" />
+    <origin xyz="0 0 0" rpy="${tY*PI/2} 0 0" />
     <mass value="${wheelMass}"/>
     <cylinder_inertia m="${wheelMass}" r="${wheelRadius}" h="${wheelWidth}"/>
   </inertial>
 </link>
-<gazebo reference="${lr}_wheel">
-  <mu1 value="200.0"/>
-  <mu2 value="100.0"/>
-  <kp value="10000000.0" />
+<!-- <gazebo reference="${lr}_wheel">
+  <mu1 value="1.0"/>
+  <mu2 value="1.0"/>
+  <kp value="100000.0" />
   <kd value="1.0" />
-  <fdir1 value="1 0 0"/>
   <material>Gazebo/Black</material>
-</gazebo>
+</gazebo>  -->
   <joint name="${lr}_wheel_joint" type="continuous">
     <axis xyz="0 1 0" rpy="0 0 0" />
@@ -76,6 +75,6 @@
     <child link="${lr}_wheel"/>
     <origin xyz="0 ${tY*(motorWidth/2+wheelWidth/2)} 0" rpy="0 0 0"/>
-    <limit effort="100" velocity="100"/>
-    <joint_properties damping="0.0" friction="0.0"/>
+    <!--<limit effort="100" velocity="100"/>
+    <joint_properties damping="0.0" friction="0.0"/>-->
   </joint>
 <transmission name="${lr}_trans">
@@ -84,5 +83,5 @@
     <hardwareInterface>hardware_interface/VelocityJointInterface</hardwareInterface>
   </joint>
-  <actuator name="${lr}Motor">
+  <actuator name="${lr}_motor">
     <mechanicalReduction>1</mechanicalReduction>
   </actuator>

Commit message: interface compiled

File: bilbot_description/urdf/bilbot.xacro (robot description, xacro)
@@ -91,12 +91,12 @@
   </inertial>
 </link>
-<!-- <joint name="battery_joint" type="fixed">
+<joint name="battery_joint" type="fixed">
   <parent link="chassis"/>
   <child link="battery"/>
-  <origin xyz="${batteryOffset} 0 ${chassisHeight/2}" rpy="0 0 0"/>
+  <origin xyz="0 0 ${chassisHeight/2 + batteryHeight/2}" rpy="0 0 0"/>
 </joint>
 <link name="battery">
   <collision>
-    <origin xyz="0 0 ${batteryHeight/2}" rpy="0 0 0"/>
+    <origin xyz="0 0 0" rpy="0 0 0"/>
     <geometry>
       <box size="${batteryLength} ${batteryWidth} ${batteryHeight}"/>
@@ -104,5 +104,5 @@
   </collision>
   <visual>
-    <origin xyz="0 0 ${batteryHeight/2}" rpy="0 0 0"/>
+    <origin xyz="0 0 0" rpy="0 0 0"/>
     <geometry>
       <box size="${batteryLength} ${batteryWidth} ${batteryHeight}"/>
@@ -163,5 +163,5 @@
   </inertial>
 </link>
-<joint name="raspberrypi_joint" type="fixed">
+<!-- <joint name="raspberrypi_joint" type="fixed">
   <parent link="layer"/>
   <child link="raspberrypi"/>
@@ -215,9 +215,9 @@
 <xacro:wheel lr="right" tY="1"/>
 <xacro:wheel lr="left" tY="-1"/>
-<!-- <xacro:gripper/>
-<xacro:support lr="left" fb="front" tY="1" tX="1"/>
+<!-- <xacro:gripper/> -->
+<!-- <xacro:support lr="left" fb="front" tY="1" tX="1"/>
 <xacro:support lr="right" fb="front" tY="-1" tX="1"/>
 <xacro:support lr="left" fb="back" tY="1" tX="-1"/>
-<xacro:support lr="right" fb="back" tY="-1" tX="-1"/>
+<xacro:support lr="right" fb="back" tY="-1" tX="-1"/> -->
  <joint name="camera_joint" type="fixed">
   <parent link="front"/>
@@ -319,4 +319,4 @@
       <box_inertia m="${laserMass}" x="${laserWidth}" y="${laserLength}" z="${laserHeight}" />
     </inertial>
-  </link> -->
+  </link>
 </robot>

File: bilbot_description/urdf/macros.xacro (robot description, xacro)
@@ -63,5 +63,5 @@
   </inertial>
 </link>
-<!-- <gazebo reference="${lr}_wheel">
+<gazebo reference="${lr}_wheel">
   <mu1 value="1.0"/>
   <mu2 value="1.0"/>
@@ -69,5 +69,5 @@
   <kd value="1.0" />
   <material>Gazebo/Black</material>
-</gazebo>  -->
+</gazebo>
   <joint name="${lr}_wheel_joint" type="continuous">
     <axis xyz="0 1 0" rpy="0 0 0" />
